Commit message: updated model

File: robot_description/urdf/robot_description.urdf (robot description, URDF)
Before this commit: robot robot_description, 16 links, 15 joints
Links:
- removed link base1_link
- removed link ramie_rot
- removed link ramie_rot2
- removed link ramie_rot_base2
- added link base_link, mass 0.65449; collision mesh filename=package://robot_description/meshes/base_link.STL; visual mesh filename=package://robot_description/meshes/base_link.STL
- added link base_up, mass 0.659790295336421; collision mesh filename=package://robot_description/meshes/base_up.STL; visual mesh filename=package://robot_description/meshes/base_up.STL
- added link ramie1_sworzen, mass 0.080353; collision mesh filename=package://robot_description/meshes/ramie1_sworzen.STL; visual mesh filename=package://robot_description/meshes/ramie1_sworzen.STL
- added link ramie2_sworzen, mass 0.0803528752062073; collision mesh filename=package://robot_description/meshes/ramie2_sworzen.STL; visual mesh filename=package://robot_description/meshes/ramie2_sworzen.STL
- added link ramie3_sworzen, mass 0.0803528752062073; collision mesh filename=package://robot_description/meshes/ramie3_sworzen.STL; visual mesh filename=package://robot_description/meshes/ramie3_sworzen.STL
- added link ramie_gora, mass 0.65979029533642; collision mesh filename=package://robot_description/meshes/ramie_gora.STL; visual mesh filename=package://robot_description/meshes/ramie_gora.STL
- added link ramie_ruch1, mass 0.0824025158054101; collision mesh filename=package://robot_description/meshes/ramie_ruch1.STL; visual mesh filename=package://robot_description/meshes/ramie_ruch1.STL
- added link ramie_ruch2, mass 0.0871028752062767; collision mesh filename=package://robot_description/meshes/ramie_ruch2.STL; visual mesh filename=package://robot_description/meshes/ramie_ruch2.STL
- added link sworzen1, mass 0.66332; collision mesh filename=package://robot_description/meshes/sworzen1.STL; visual mesh filename=package://robot_description/meshes/sworzen1.STL
- added link sworzen2, mass 0.663324587071708; collision mesh filename=package://robot_description/meshes/sworzen2.STL; visual mesh filename=package://robot_description/meshes/sworzen2.STL
- added link sworzen3, mass 0.663324587071708; collision mesh filename=package://robot_description/meshes/sworzen3.STL; visual mesh filename=package://robot_description/meshes/sworzen3.STL
- added link sworzen4, mass 0.66332458707171; collision mesh filename=package://robot_description/meshes/sworzen4.STL; visual mesh filename=package://robot_description/meshes/sworzen4.STL
- added link sworzen5, mass 0.66332458707171; collision mesh filename=package://robot_description/meshes/sworzen5.STL; visual mesh filename=package://robot_description/meshes/sworzen5.STL
- added link sworzen6, mass 0.66332458707171; collision mesh filename=package://robot_description/meshes/sworzen6.STL; visual mesh filename=package://robot_description/meshes/sworzen6.STL
- added link sworzen_ramie4, mass 0.0803528752062073; collision mesh filename=package://robot_description/meshes/sworzen_ramie4.STL; visual mesh filename=package://robot_description/meshes/sworzen_ramie4.STL
- added link sworzen_ramie5, mass 0.080353; collision mesh filename=package://robot_description/meshes/sworzen_ramie5.STL; visual mesh filename=package://robot_description/meshes/sworzen_ramie5.STL
- added link sworzen_ramie6, mass 0.0803528752062072; collision mesh filename=package://robot_description/meshes/sworzen_ramie6.STL; visual mesh filename=package://robot_description/meshes/sworzen_ramie6.STL
- added link sworzen_ramie_ruch, mass 0.0824025158054101; collision mesh filename=package://robot_description/meshes/sworzen_ramie_ruch.STL; visual mesh filename=package://robot_description/meshes/sworzen_ramie_ruch.STL
- added link sworzen_ramie_ruch2, mass 0.0871028752062767; collision mesh filename=package://robot_description/meshes/sworzen_ramie_ruch2.STL; visual mesh filename=package://robot_description/meshes/sworzen_ramie_ruch2.STL
- link kolo1: mass 0.110515551952779 -> 0.040766
- link kolo2: mass 0.110515551952779 -> 0.0407655519524368
- link kolo3: mass 0.110515551952779 -> 0.0407655519524369
- link kolo4: mass 0.110515551952779 -> 0.040766
- link kolo5: mass 0.110515551952779 -> 0.040766
- link kolo6: mass 0.11052 -> 0.0407655519524368
- link ramie1: mass 0.72954 -> 0.083887
- link ramie2: mass 0.729540295336762 -> 0.0838871669414958
- link ramie3: mass 0.729540295336762 -> 0.0838871669414958
- link ramie4: mass 0.729540295336761 -> 0.0838871669414958
- link ramie5: mass 0.729540295336761 -> 0.0838871669414958
- link ramie6: mass 0.729540295336761 -> 0.0838871669414958
Joints:
- removed joint ramie_rot2_joint
- removed joint ramie_rot_base2_joint
- removed joint ramie_rot_joint
- added joint base_up_joint: type revolute, parent sworzen_ramie_ruch2, child base_up, origin xyz=0.015 0.1 -0.015 rpy=-2.2204E-16 -9.7838E-16 -2.9613, axis 0 0 0, limit lower=-1.57 upper=1.57 effort=0 velocity=0
- added joint ramie1_sworzen_joint: type revolute, parent ramie1, child ramie1_sworzen, origin xyz=0.005881 0.013799 0.025 rpy=-3.3307E-16 -9.992E-16 -1.9737, axis 0 0 0, limit lower=-1.57 upper=1.57 effort=0 velocity=0
- added joint ramie2_sworzen_joint: type revolute, parent ramie2, child ramie2_sworzen, origin xyz=0.0020565 0.014858 0.025 rpy=4.4409E-16 -1.0547E-15 -1.7083, axis 0 0 0, limit lower=-1.57 upper=1.57 effort=0 velocity=0
- added joint ramie3_sworzen_joint: type revolute, parent ramie3, child ramie3_sworzen, origin xyz=0.0074468 -0.013021 0.025 rpy=3.1416 1.1328E-15 2.0903, axis 0 0 0, limit lower=-1.57 upper=1.57 effort=0 velocity=0
- added joint ramie_gora_joint: type fixed, parent base_link, child ramie_gora, origin xyz=0.078656 0.0046714 -0.033295 rpy=-1.0935 -1.209 1.6195, axis 0 0 0
- added joint ramie_ruch1_joint: type revolute, parent ramie_gora, child ramie_ruch1, origin xyz=0 0.03 -0.015 rpy=3.0531E-16 -9.4369E-16 -2.341, axis 0 0 0, limit lower=-1.57 upper=1.57 effort=0 velocity=0
- added joint ramie_ruch2_joint: type revolute, parent sworzen_ramie_ruch, child ramie_ruch2, origin xyz=0 0 0 rpy=-5.5511E-17 0 -5.5511E-17, axis 0 0 0, limit lower=-1.57 upper=1.57 effort=0 velocity=0
- added joint sworzen1_joint: type revolute, parent base_link, child sworzen1, origin xyz=0.078656 0.0046714 -0.033295 rpy=-1.0935 -1.209 1.6195, axis 0 0 0, limit lower=-1.57 upper=1.57 effort=0 velocity=0
- added joint sworzen2_joint: type revolute, parent base_link, child sworzen2, origin xyz=0.078656 0.0046714 -0.033295 rpy=-1.0935 -1.209 1.6195, axis 0 0 0, limit lower=-1.57 upper=1.57 effort=0 velocity=0
- added joint sworzen3_joint: type revolute, parent base_link, child sworzen3, origin xyz=0.078656 0.0046714 -0.033295 rpy=-1.0935 -1.209 1.6195, axis 0 0 0, limit lower=-1.57 upper=1.57 effort=0 velocity=0
- added joint sworzen4_joint: type revolute, parent base_up, child sworzen4, origin xyz=-0.0053809 -0.029513 0.015 rpy=0.18034 -1.5708 0, axis 0 0 0, limit lower=-1.57 upper=1.57 effort=0 velocity=0
- added joint sworzen5_joint: type revolute, parent base_up, child sworzen5, origin xyz=-0.0053809 -0.029513 0.015 rpy=0.18034 -1.5708 0, axis 0 0 0, limit lower=-1.57 upper=1.57 effort=0 velocity=0
- added joint sworzen6_joint: type revolute, parent base_up, child sworzen6, origin xyz=-0.0053809 -0.029513 0.015 rpy=0.18034 -1.5708 0, axis 0 0 0, limit lower=-1.57 upper=1.57 effort=0 velocity=0
- added joint sworzen_ramie4_joint: type revolute, parent ramie4, child sworzen_ramie4, origin xyz=0.012416 0.0084172 0.025 rpy=-3.1416 -1.3711E-14 -2.5458, axis 0 0 0, limit lower=-1.57 upper=1.57 effort=0 velocity=0
- added joint sworzen_ramie5_joint: type revolute, parent ramie5, child sworzen_ramie5, origin xyz=0.099571 0.0092516 0.01 rpy=-1.1137E-15 -6.1062E-15 -2.4427, axis 0 0 0, limit lower=-1.57 upper=1.57 effort=0 velocity=0
- added joint sworzen_ramie6_joint: type revolute, parent ramie6, child sworzen_ramie6, origin xyz=0.014217 -0.004782 0.025 rpy=-3.1416 -3.8441E-15 2.8171, axis 0 0 0, limit lower=-1.57 upper=1.57 effort=0 velocity=0
- added joint sworzen_ramie_ruch2_joint: type revolute, parent ramie_ruch2, child sworzen_ramie_ruch2, origin xyz=0.0009318 -0.014971 0.015 rpy=3.7192E-15 3.4694E-16 1.633, axis 0 0 0, limit lower=-1.57 upper=1.57 effort=0 velocity=0
- added joint sworzen_ramie_ruch_joint: type revolute, parent ramie_ruch1, child sworzen_ramie_ruch, origin xyz=-0.070166 -0.072813 0.015 rpy=1.5708 -0.22145 0.95279, axis 0 0 0, limit lower=-1.57 upper=1.57 effort=0 velocity=0
- joint kolo1_joint: origin xyz=-0.087213 -0.0078411 0 rpy=-3.1416 -1.1685E-14 2.5915 -> xyz=0.015 0.1 -0.0075 rpy=1.2654 -1.5708 0; parent ramie1 -> ramie1_sworzen; type fixed -> continuous
- joint kolo2_joint: origin xyz=0.041089 0.095135 -0.056168 rpy=0.84288 0.5236 -3.1416 -> xyz=0.015 0.1 -0.015 rpy=-6.4948E-15 1.3323E-15 -2.0595; parent ramie2 -> ramie2_sworzen; type fixed -> continuous
- joint kolo3_joint: origin xyz=0.055717 0.0097094 0.096504 rpy=-2.2991 0.72098 -2.1029 -> xyz=0.015 0.1 0.015 rpy=-3.1416 3.1572E-16 0.26592; parent ramie3 -> ramie3_sworzen; type fixed -> continuous
- joint kolo4_joint: origin xyz=0.044738 0.010688 -0.077488 rpy=2.2518 0.65307 -1.1133 -> xyz=0.015 0.1 0.015 rpy=3.1416 3.6082E-16 -0.13282; parent ramie4 -> sworzen_ramie4; type fixed -> continuous
- joint kolo5_joint: origin xyz=-0.08712 0.007688 0 rpy=1.1102E-16 -6.1062E-16 -2.6035 -> xyz=0 0 0 rpy=-3.4694E-17 0 -2.7756E-17; parent ramie5 -> sworzen_ramie5; type fixed -> continuous
- joint kolo6_joint: origin xyz=0.043799 0.0084384 0.075863 rpy=-2.3692 -0.79805 -0.93708 -> xyz=0.015 0.1 -0.015 rpy=8.743E-16 7.2164E-16 -2.1766; parent ramie6 -> sworzen_ramie6; type fixed -> continuous
- joint ramie1_joint: limit lower=1.0472 upper=3.1416 effort=0 velocity=0 -> lower=-1.57 upper=1.57 effort=0 velocity=0; origin xyz=-0.014472 0.21014 -0.15632 rpy=-1.6144 1.0405 -1.3565 -> xyz=0.028349 0 0.099103 rpy=-2.3896 0.81672 -2.2328; parent base1_link -> sworzen1
- joint ramie2_joint: limit lower=1.0472 upper=3.1416 effort=0 velocity=0 -> lower=-1.57 upper=1.57 effort=0 velocity=0; origin xyz=-0.014472 0.21014 -0.15632 rpy=-1.6144 1.0405 -1.3565 -> xyz=-0.1 0 -0.025 rpy=3.8858E-16 2.498E-16 -0.89513; parent base1_link -> sworzen2
- joint ramie3_joint: limit lower=1.0472 upper=3.1416 effort=0 velocity=0 -> lower=-1.57 upper=1.57 effort=0 velocity=0; origin xyz=-0.014472 0.21014 -0.15632 rpy=-1.6144 1.0405 -1.3565 -> xyz=0.028349 0 -0.099103 rpy=-0.41636 -0.99237 -2.6557; parent base1_link -> sworzen3
- joint ramie4_joint: limit lower=1.0472 upper=3.1416 effort=0 velocity=0 -> lower=-1.57 upper=1.57 effort=0 velocity=0; origin xyz=0.020446 -0.029502 0 rpy=3.1416 0 -2.959 -> xyz=-0.1 0 -0.025 rpy=2.38E-15 -8.0491E-16 -1.1458; parent ramie_rot_base2 -> sworzen4
- joint ramie5_joint: limit lower=1.0472 upper=3.1416 effort=0 velocity=0 -> lower=-1.57 upper=1.57 effort=0 velocity=0; origin xyz=0.020446 -0.029502 0 rpy=3.1416 0 -2.959 -> xyz=0.028349 0 0.099103 rpy=2.2611 0.66778 2.0435; parent ramie_rot_base2 -> sworzen5
- joint ramie6_joint: limit lower=1.0472 upper=3.1416 effort=0 velocity=0 -> lower=-1.57 upper=1.57 effort=0 velocity=0; origin xyz=0.020446 -0.029502 0 rpy=3.1416 0 -2.959 -> xyz=0.028349 0 -0.099103 rpy=0.80073 0.76958 0.97718; parent ramie_rot_base2 -> sworzen6
